Commit message: Synchronization issue solved

File: arm_urdf_moveit_config/config/ArmPlate.ros2_control.xacro (robot description, xacro)
@@ -3,10 +3,4 @@
     <xacro:macro name="ArmPlate_ros2_control" params="name initial_positions_file">
         <xacro:property name="initial_positions" value="${load_yaml(initial_positions_file)['initial_positions']}"/>
-        <!-- <ros2_control name="${name}" type="system">
-            <hardware>
-                <plugin>mock_components/GenericSystem</plugin>
-            </hardware>
-            </joint>
-        </ros2_control> -->
         <ros2_control name="Servo" type="system">
             <hardware>
