Commit message: Modified urdf and stepper

File: arm_urdf/urdf/ArmPlate.xacro (robot description, xacro)
@@ -197,10 +197,16 @@
         <child link="grasp_frame" />
     </joint>
-    <joint name="Base_link1-v1_Revolute-1" type="continuous">
-        <origin xyz="-0.05188764 -0.052144760000000005 0.01" rpy="3.141592653589793 -0.0 0.594" />
-        <parent link="Base_link1-v1" />
-        <child link="2ndDOFDDD-v1" />
-        <axis xyz="0.0 -1.158152704299605e-16 1.0" />
-    </joint>
+<joint name="Base_link1-v1_Revolute-1" type="revolute">
+    <origin xyz="-0.05188764 -0.052144760000000005 0.01"
+            rpy="3.141592653589793 -0.0 0.594" />
+    <parent link="Base_link1-v1" />
+    <child link="2ndDOFDDD-v1" />
+    <axis xyz="0.0 -1.158152704299605e-16 1.0" />
+    <limit
+        lower="0.0"
+        upper="6.283185307"
+        effort="10.0"
+        velocity="1.0" />
+</joint>
     <joint name="2ndDOFDDD-v1_Revolute-8" type="revolute">
         <origin xyz="0.052840300000000937 -0.004111319999999985 -0.13483788000000002" rpy="1.5707963267948974 1.5707963267948828 -1.6484463606696926" />
@@ -233,9 +239,9 @@
         <child link="gripperHousing-v2" />
         <axis xyz="0.0 -2.21569993751437e-32 1.0" />
-        <limit
-        lower="-3.14159"
-        upper="2.0944"
-        effort="10"
-        velocity="2.0" />
+    <limit
+        lower="0.0"
+        upper="6.283185307"
+        effort="10.0"
+        velocity="1.0" />
     </joint>
     <joint name="gripperHousing-v2_Slider-13" type="prismatic">

Commit message: Hand working

File: arm_urdf/urdf/ArmPlate.xacro (robot description, xacro)
@@ -199,11 +199,11 @@
 <joint name="Base_link1-v1_Revolute-1" type="revolute">
     <origin xyz="-0.05188764 -0.052144760000000005 0.01"
-            rpy="3.141592653589793 -0.0 0.09" />
+            rpy="3.141592653589793 -0.0 -0.05" />
     <parent link="Base_link1-v1" />
     <child link="2ndDOFDDD-v1" />
     <axis xyz="0.0 -1.158152704299605e-16 1.0" />
     <limit
-        lower="0.0"
-        upper="6.1959188"
+        lower="0.174533"
+        upper="6.108652"
         effort="10.0"
         velocity="100.0" />

File: arm_urdf_moveit_config/config/ArmPlate.ros2_control.xacro (robot description, xacro)
@@ -3,19 +3,15 @@
     <xacro:macro name="ArmPlate_ros2_control" params="name initial_positions_file">
         <xacro:property name="initial_positions" value="${load_yaml(initial_positions_file)['initial_positions']}"/>
-        <ros2_control name="${name}" type="system">
+        <!-- <ros2_control name="${name}" type="system">
             <hardware>
                 <plugin>mock_components/GenericSystem</plugin>
             </hardware>
-            <joint name="gripperHousing-v2_Slider-13">
-                <command_interface name="position"/>
-                <state_interface name="position">
-                  <param name="initial_value">${initial_positions['gripperHousing-v2_Slider-13']}</param>
-                </state_interface>
             </joint>
-        </ros2_control>
+        </ros2_control> -->
         <ros2_control name="Servo" type="system">
             <hardware>
                 <plugin>arm_servo_controller/ArmServoHardware</plugin>
                 <param name="port">/dev/arm_servo</param>
+                <param name="gripper_id">9</param>
             </hardware>
             <!-- <hardware>
@@ -27,4 +23,11 @@
                 <state_interface name="position">
                   <param name="initial_value">${initial_positions['6Thdof-v2_Revolute-12']}</param>
+                </state_interface>
+            </joint>
+            <joint name="gripperHousing-v2_Slider-13">
+                <param name="id">9</param>
+                <command_interface name="position"/>
+                <state_interface name="position">
+                  <param name="initial_value">${initial_positions['gripperHousing-v2_Slider-13']}</param>
                 </state_interface>
             </joint>

Commit message: Working pnp

File: arm_urdf/urdf/ArmPlate.xacro (robot description, xacro)
@@ -197,16 +197,11 @@
         <child link="grasp_frame" />
     </joint>
-<joint name="Base_link1-v1_Revolute-1" type="revolute">
-    <origin xyz="-0.05188764 -0.052144760000000005 0.01"
-            rpy="3.141592653589793 -0.0 -0.05" />
-    <parent link="Base_link1-v1" />
-    <child link="2ndDOFDDD-v1" />
-    <axis xyz="0.0 -1.158152704299605e-16 1.0" />
-    <limit
-        lower="0.174533"
-        upper="6.108652"
-        effort="10.0"
-        velocity="100.0" />
-</joint>
+    <joint name="Base_link1-v1_Revolute-1" type="revolute">
+        <origin xyz="-0.05188764 -0.052144760000000005 0.01" rpy="3.141592653589793 -0.0 -0.05" />
+        <parent link="Base_link1-v1" />
+        <child link="2ndDOFDDD-v1" />
+        <axis xyz="0.0 -1.158152704299605e-16 1.0" />
+        <limit lower="0.174533" upper="6.108652" effort="10.0" velocity="100.0" />
+    </joint>
     <joint name="2ndDOFDDD-v1_Revolute-8" type="revolute">
         <origin xyz="0.052840300000000937 -0.004111319999999985 -0.13483788000000002" rpy="1.5707963267948974 1.5707963267948828 -1.6484463606696926" />
