Commit message: Full urdf, new config files

File: arm_urdf/urdf/ArmPlate.xacro (robot description, xacro)
@@ -1,190 +1,362 @@
 <?xml version='1.0' encoding='utf-8'?>
 <robot name="ArmPlate">
-    <link name="world"/>
-    <joint name="base_to_world" type="fixed">
-        <parent link="world" />
-        <child link="Base_link1-v1" />
-    </joint>
-    <link name="Base_link1-v1">
-        <inertial>
-            <origin xyz="-0.0674024747578498 -0.052144759691377905 0.001871879485998631" rpy="0.0 0.0 0.0" />
-            <mass value="4.311969816496875" />
-            <inertia ixx="0.03729401814426159" iyy="0.028233182216333773" izz="0.06539104879017638" ixy="-3.479855292809475e-15" iyz="1.0668549377257364e-16" ixz="-0.00020885219602048547" />
-        </inertial>
-        <visual name="Base_link1-v1_visual">
+    <link name="5thDof_mnt-v2">
+        <inertial>
+            <origin xyz="0.012732324690562784 0.031437498134228435 -0.0003069334959384307" rpy="0.0 -0.0 -1.4025374347724758e-59" />
+            <mass value="0.7682943067467453" />
+            <inertia ixx="0.000535840458777137" iyy="0.0008753213536334542" izz="0.001103925893107316" ixy="-0.00016097281530438878" iyz="2.184664611465381e-06" ixz="1.1367846554491412e-05" />
+        </inertial>
+        <visual name="5thDof_mnt-v2_visual">
+            <origin xyz="-0.06150135283187986 0.041275362887439895 2.5317682528225306e-09" rpy="-1.570796326794906 9.156666191836695e-15 1.5744533391479172" />
+            <geometry>
+                <mesh filename="package://arm_urdf/meshes/5thDof_mnt-v2.stl" scale="0.001 0.001 0.001" />
+            </geometry>
+        </visual>
+        <collision name="5thDof_mnt-v2_collision">
+            <origin xyz="-0.06150135283187986 0.041275362887439895 2.5317682528225306e-09" rpy="-1.570796326794906 9.156666191836695e-15 1.5744533391479172" />
+            <geometry>
+                <mesh filename="package://arm_urdf/meshes/5thDof_mnt-v2.stl" scale="0.001 0.001 0.001" />
+            </geometry>
+        </collision>
+    </link>
+    <link name="6Thdof-v2">
+        <inertial>
+            <origin xyz="-0.008352271711918942 0.031354612679946714 -2.1198788677914137e-05" rpy="0.0 -0.0 0.0" />
+            <mass value="0.8639927133401125" />
+            <inertia ixx="0.0009570909963230179" iyy="0.0002912622479420493" izz="0.0009228135461331055" ixy="5.0224618618324723e-05" iyz="1.3662637325731475e-05" ixz="-8.244285327335676e-08" />
+        </inertial>
+        <visual name="6Thdof-v2_visual">
+            <origin xyz="-0.010299810307640645 0.08196288452277116 -0.013749997468232316" rpy="-1.5707963267949052 -9.411824927776451e-15 0.003657012352839137" />
+            <geometry>
+                <mesh filename="package://arm_urdf/meshes/6Thdof-v2.stl" scale="0.001 0.001 0.001" />
+            </geometry>
+        </visual>
+        <collision name="6Thdof-v2_collision">
+            <origin xyz="-0.010299810307640645 0.08196288452277116 -0.013749997468232316" rpy="-1.5707963267949052 -9.411824927776451e-15 0.003657012352839137" />
+            <geometry>
+                <mesh filename="package://arm_urdf/meshes/6Thdof-v2.stl" scale="0.001 0.001 0.001" />
+            </geometry>
+        </collision>
+    </link>
+    <link name="redassm-v1">
+        <inertial>
+            <origin xyz="0.0045480904541335574 -0.008359528801030676 0.10098035514768636" rpy="0.0 -0.0 0.0" />
+            <mass value="6.794045956021914" />
+            <inertia ixx="0.04847097589923233" iyy="0.051084808654606795" izz="0.02583120358184199" ixy="-0.0005049440216612079" iyz="0.0009392673544488904" ixz="0.000615655195551375" />
+        </inertial>
+        <visual name="redassm-v1_visual">
+            <origin xyz="4.456090927362766e-09 1.018317314915862e-09 0.009000003253548154" rpy="8.388603136835838e-15 -7.460303902010976e-15 -0.07399302152178323" />
+            <geometry>
+                <mesh filename="package://arm_urdf/meshes/redassm-v1.stl" scale="0.001 0.001 0.001" />
+            </geometry>
+        </visual>
+        <collision name="redassm-v1_collision">
+            <origin xyz="4.456090927362766e-09 1.018317314915862e-09 0.009000003253548154" rpy="8.388603136835838e-15 -7.460303902010976e-15 -0.07399302152178323" />
+            <geometry>
+                <mesh filename="package://arm_urdf/meshes/redassm-v1.stl" scale="0.001 0.001 0.001" />
+            </geometry>
+        </collision>
+    </link>
+    <link name="newUpp-v1">
+        <inertial>
+            <origin xyz="-0.0018373155063777168 -0.09523668822442201 0.13827055961369247" rpy="0.0 -0.0 3.94430452610506e-31" />
+            <mass value="3.8828589051011537" />
+            <inertia ixx="0.05707845804840468" iyy="0.032921156778058486" izz="0.02426709686098271" ixy="0.00014947243101293955" iyz="-0.00020923786947107248" ixz="-6.027251910115146e-06" />
+        </inertial>
+        <visual name="newUpp-v1_visual">
+            <origin xyz="-3.253549269999212e-09 -0.030880127170425417 0.18991252867308034" rpy="1.5707963267948748 2.962977085907427e-13 -1.5707963267949003" />
+            <geometry>
+                <mesh filename="package://arm_urdf/meshes/newUpp-v1.stl" scale="0.001 0.001 0.001" />
+            </geometry>
+        </visual>
+        <collision name="newUpp-v1_collision">
+            <origin xyz="-3.253549269999212e-09 -0.030880127170425417 0.18991252867308034" rpy="1.5707963267948748 2.962977085907427e-13 -1.5707963267949003" />
+            <geometry>
+                <mesh filename="package://arm_urdf/meshes/newUpp-v1.stl" scale="0.001 0.001 0.001" />
+            </geometry>
+        </collision>
+    </link>
+    <link name="Component9-v4">
+        <inertial>
+            <origin xyz="0.0014195000758181731 0.0003605891225194885 0.10432232092473005" rpy="0.0 0.0 0.0" />
+            <mass value="11.219161423050371" />
+            <inertia ixx="0.23259258909874736" iyy="0.3481854187292448" izz="0.5733793475673593" ixy="0.0009456976306902002" iyz="-3.711339435333852e-05" ixz="-0.0001461600503889675" />
+        </inertial>
+        <visual name="Component9-v4_visual">
             <origin xyz="0.0 0.0 0.0" rpy="0.0 0.0 0.0" />
             <geometry>
-                <mesh filename="package://arm_urdf/meshes/Base_link1-v1.stl" scale="0.001 0.001 0.001" />
-            </geometry>
-        </visual>
-        <collision name="Base_link1-v1_collision">
+                <mesh filename="package://arm_urdf/meshes/Component9-v4.stl" scale="0.001 0.001 0.001" />
+            </geometry>
+        </visual>
+        <collision name="Component9-v4_collision">
             <origin xyz="0.0 0.0 0.0" rpy="0.0 0.0 0.0" />
             <geometry>
-                <mesh filename="package://arm_urdf/meshes/Base_link1-v1.stl" scale="0.001 0.001 0.001" />
-            </geometry>
-        </collision>
-    </link>
-    <link name="2ndDOFDDD-v1">
-        <inertial>
-            <origin xyz="0.005563007183593101 0.008083968084292402 -0.10431093233027892" rpy="0.0 -0.0 0.0" />
-            <mass value="6.914197067582951" />
-            <inertia ixx="0.0489503398990333" iyy="0.05164846688679926" izz="0.026188561835283307" ixy="0.000744724254469125" iyz="0.0009319574397850192" ixz="-0.00045704067111378735" />
-        </inertial>
-        <!-- <visual name="2ndDOFDDD-v1_visual">
-            <origin xyz="1.62650033885825e-09 -3.0861703415041576e-10 -0.011999999999999664" rpy="-3.141592653589793 -2.028647007485838e-62 1.7516230804060213e-46" />
-            <geometry>
-                <mesh filename="package://arm_urdf/meshes/2ndDOFDDD-v1.stl" scale="0.001 0.001 0.001" />
-            </geometry>
-        </visual>
-        <collision name="2ndDOFDDD-v1_collision">
-            <origin xyz="1.62650033885825e-09 -3.0861703415041576e-10 -0.011999999999999664" rpy="-3.141592653589793 -2.028647007485838e-62 1.7516230804060213e-46" />
-            <geometry>
-                <mesh filename="package://arm_urdf/meshes/2ndDOFDDD-v1.stl" scale="0.001 0.001 0.001" />
-            </geometry>
-        </collision> -->
-       <visual>
-            <origin xyz="0 0 -0.08" rpy="0 0 0"/>
-            <geometry>
-            <box size="0.1 0.1 0.2"/> <!-- x y z in meters -->
-            </geometry>
-        </visual>
-        <!-- Collision geometry -->
-        <collision>
-            <origin xyz="0 0 -0.08" rpy="0 0 0"/>
-            <geometry>
-            <box size="0.1 0.1 0.2"/>
-            </geometry>
-        </collision>
-    </link>
-    <link name="lnk1assm-v2">
-        <inertial>
-            <origin xyz="-0.002591598973958833 -0.23584751583887864 -0.00539988945227305" rpy="0.0 1.3877787807823214e-17 -1.5777218104420236e-30" />
-            <mass value="2.0414167169593447" />
-            <inertia ixx="0.029664413351168283" iyy="0.0017505470451872956" izz="0.02962243298274335" ixy="-0.00029616879202136004" iyz="0.0015603149109663106" ixz="2.540746428059758e-05" />
-        </inertial>
-        <visual name="lnk1assm-v2_visual">
-            <origin xyz="-0.003921107309494927 -0.34147748775887143 0.08610000077174858" rpy="1.0011067892201222e-15 2.63677968348484e-16 1.0432232103974771e-16" />
-            <geometry>
-                <mesh filename="package://arm_urdf/meshes/lnk1assm-v2.stl" scale="0.001 0.001 0.001" />
-            </geometry>
-        </visual>
-        <collision name="lnk1assm-v2_collision">
-            <origin xyz="-0.003921107309494927 -0.34147748775887143 0.08610000077174858" rpy="1.0011067892201222e-15 2.63677968348484e-16 1.0432232103974771e-16" />
-            <geometry>
-                <mesh filename="package://arm_urdf/meshes/lnk1assm-v2.stl" scale="0.001 0.001 0.001" />
-            </geometry>
-        </collision>
-    </link>
-    <link name="lnk2_assm-v2">
-        <inertial>
-            <origin xyz="0.015287483405147686 0.0015469235286940375 0.14314076456091882" rpy="0.0 -2.802596928649634e-45 7.718750464542261e-60" />
-            <mass value="1.6041672165297656" />
-            <inertia ixx="0.011935327683088248" iyy="0.011817416915501418" izz="0.001112072658466317" ixy="-1.4881667141780628e-06" iyz="-0.0001166157499106618" ixz="-0.0010845287768283282" />
-        </inertial>
-        <visual name="lnk2_assm-v2_visual">
-            <origin xyz="0.03287283838328484 0.003560737736243089 0.2818374324484128" rpy="-1.4080220534306864e-15 -1.059118750771804e-14 -1.4931462929201005" />
-            <geometry>
-                <mesh filename="package://arm_urdf/meshes/lnk2_assm-v2.stl" scale="0.001 0.001 0.001" />
-            </geometry>
-        </visual>
-        <collision name="lnk2_assm-v2_collision">
-            <origin xyz="0.03287283838328484 0.003560737736243089 0.2818374324484128" rpy="-1.4080220534306864e-15 -1.059118750771804e-14 -1.4931462929201005" />
-            <geometry>
-                <mesh filename="package://arm_urdf/meshes/lnk2_assm-v2.stl" scale="0.001 0.001 0.001" />
-            </geometry>
-        </collision>
-    </link>
-    <link name="5thDof_mnt-v2">
-        <inertial>
-            <origin xyz="-0.012784684069178872 -0.0013025970291178357 0.031390730609038686" rpy="0.0 -0.0 0.0" />
-            <mass value="0.7682943067467453" />
-            <inertia ixx="0.0005398526790914571" iyy="0.001098740864250658" izz="0.000876494162175584" ixy="-5.5264308595074155e-05" iyz="1.4526969696712633e-05" ixz="0.00015907949467902638" />
-        </inertial>
-        <visual name="5thDof_mnt-v2_visual">
-            <origin xyz="0.06116513562152025 0.004759041505515995 0.04150000244841479" rpy="-3.063942619714997 -1.5707963267948506 0" />
-            <geometry>
-                <mesh filename="package://arm_urdf/meshes/5thDof_mnt-v2.stl" scale="0.001 0.001 0.001" />
-            </geometry>
-        </visual>
-        <collision name="5thDof_mnt-v2_collision">
-            <origin xyz="0.06116513562152025 0.004759041505515995 0.04150000244841479" rpy="-3.063942619714997 -1.5707963267948506 0" />
-            <geometry>
-                <mesh filename="package://arm_urdf/meshes/5thDof_mnt-v2.stl" scale="0.001 0.001 0.001" />
-            </geometry>
-        </collision>
-    </link>
-    <link name="6Thdof-v2">
-        <inertial>
-            <origin xyz="0.008214367551119024 0.0006178674357249214 0.031384946859303826" rpy="-2.2420775429197073e-44 -0.0 0.0" />
-            <mass value="0.8639927133401125" />
-            <inertia ixx="0.0009572359903424752" iyy="0.0009230269883602205" izz="0.0002909038116962609" ixy="2.710767043214595e-06" iyz="9.914638568871148e-06" ixz="-4.8704209516635046e-05" />
-        </inertial>
-        <visual name="6Thdof-v2_visual">
-            <origin xyz="0.011036478474497909 -0.012932846063207827 0.08200000244841477" rpy="4.266020662176333e-15 4.485125411027998e-14 -3.0639426197149975" />
-            <geometry>
-                <mesh filename="package://arm_urdf/meshes/6Thdof-v2.stl" scale="0.001 0.001 0.001" />
-            </geometry>
-        </visual>
-        <collision name="6Thdof-v2_collision">
-            <origin xyz="0.011036478474497909 -0.012932846063207827 0.08200000244841477" rpy="4.266020662176333e-15 4.485125411027998e-14 -3.0639426197149975" />
-            <geometry>
-                <mesh filename="package://arm_urdf/meshes/6Thdof-v2.stl" scale="0.001 0.001 0.001" />
-            </geometry>
-        </collision>
-    </link>
-    <link name="gripperHousing-v2">
-        <inertial>
-            <origin xyz="-0.00013921429310007394 0.001855694220722368 0.047786878393741856" rpy="0.0 -0.0 0.0" />
-            <mass value="0.5576326934437552" />
-            <inertia ixx="0.0004695146364697145" iyy="0.0008816687160502767" izz="0.0006167594787314344" ixy="-3.232159477185512e-05" iyz="-1.2242098957490621e-05" ixz="9.183742992122149e-07" />
-        </inertial>
-        <visual name="gripperHousing-v2_visual">
-            <origin xyz="-1.525502200117046e-09 3.936792145609047e-09 2.4484144489633764e-09" rpy="-4.266020662176041e-15 -2.0620936462850397e-14 0.07765003387479581" />
-            <geometry>
-                <mesh filename="package://arm_urdf/meshes/gripperHousing-v2.stl" scale="0.001 0.001 0.001" />
-            </geometry>
-        </visual>
-        <collision name="gripperHousing-v2_collision">
-            <origin xyz="-1.525502200117046e-09 3.936792145609047e-09 2.4484144489633764e-09" rpy="-4.266020662176041e-15 -2.0620936462850397e-14 0.07765003387479581" />
-            <geometry>
-                <mesh filename="package://arm_urdf/meshes/gripperHousing-v2.stl" scale="0.001 0.001 0.001" />
-            </geometry>
-        </collision>
-    </link>
-    <link name="left_H-v1">
-        <inertial>
-            <origin xyz="-0.03857920530896109 -0.002507519809183858 0.0001992428471497476" rpy="-4.121466071543581e-45 -0.0 0.0" />
-            <mass value="0.4330027264168371" />
-            <inertia ixx="0.0001531814190167935" iyy="0.0003859475340479146" izz="0.00034050173036892506" ixy="-1.8463860142345745e-05" iyz="1.4471313147474644e-05" ixz="4.1220378661202906e-05" />
-        </inertial>
-        <visual name="left_H-v1_visual">
-            <origin xyz="0.03539594370174484 -0.026115815402647638 -0.029483865374257602" rpy="-2.6340835845626366e-13 1.4931462929201007 -1.570796326795163" />
-            <geometry>
-                <mesh filename="package://arm_urdf/meshes/left_H-v1.stl" scale="0.001 0.001 0.001" />
-            </geometry>
-        </visual>
-        <collision name="left_H-v1_collision">
-            <origin xyz="0.03539594370174484 -0.026115815402647638 -0.029483865374257602" rpy="-2.6340835845626366e-13 1.4931462929201007 -1.570796326795163" />
-            <geometry>
-                <mesh filename="package://arm_urdf/meshes/left_H-v1.stl" scale="0.001 0.001 0.001" />
-            </geometry>
-        </collision>
-    </link>
-    <link name="right_H-v1">
-        <inertial>
-            <origin xyz="0.03857921508488488 0.0025075221635958746 0.00019924149858097985" rpy="-2.9674555715114166e-45 -0.0 0.0" />
-            <mass value="0.4330027264168263" />
-            <inertia ixx="0.00015318174926833418" iyy="0.0003859473890370778" izz="0.0003405012645987804" ixy="-1.8463956405788322e-05" iyz="-1.4471222312344915e-05" ixz="-4.122038659255113e-05" />
-        </inertial>
-        <visual name="right_H-v1_visual">
-            <origin xyz="0.0014000027762429569 0.02697397988318141 -0.06071536489232356" rpy="-1.5707963267951677 -1.4931462929201007 -1.570796326794629" />
-            <geometry>
-                <mesh filename="package://arm_urdf/meshes/right_H-v1.stl" scale="0.001 0.001 0.001" />
-            </geometry>
-        </visual>
-        <collision name="right_H-v1_collision">
-            <origin xyz="0.0014000027762429569 0.02697397988318141 -0.06071536489232356" rpy="-1.5707963267951677 -1.4931462929201007 -1.570796326794629" />
-            <geometry>
-                <mesh filename="package://arm_urdf/meshes/right_H-v1.stl" scale="0.001 0.001 0.001" />
+                <mesh filename="package://arm_urdf/meshes/Component9-v4.stl" scale="0.001 0.001 0.001" />
+            </geometry>
+        </collision>
+    </link>
+    <link name="Component20">
+        <inertial>
+            <origin xyz="1.4090896272023202e-09 -3.2535519345344713e-09 0.04459999797126967" rpy="0.0 -0.0 0.0" />
+            <mass value="6.723396328206732" />
+            <inertia ixx="0.010956805237582912" iyy="0.010956805237583245" izz="0.019417168595860512" ixy="-5.551115123125783e-17" iyz="-8.382926173276683e-17" ixz="-5.043270567565005e-33" />
+        </inertial>
+        <visual name="Component20_visual">
+            <origin xyz="1.4090896627294568e-09 -3.2535520944065865e-09 0.06819999797126945" rpy="1.570796326794897 1.57079632679489 0" />
+            <geometry>
+                <mesh filename="package://arm_urdf/meshes/Component20.stl" scale="0.001 0.001 0.001" />
+            </geometry>
+        </visual>
+        <collision name="Component20_collision">
+            <origin xyz="1.4090896627294568e-09 -3.2535520944065865e-09 0.06819999797126945" rpy="1.570796326794897 1.57079632679489 0" />
+            <geometry>
+                <mesh filename="package://arm_urdf/meshes/Component20.stl" scale="0.001 0.001 0.001" />
+            </geometry>
+        </collision>
+    </link>
+    <link name="Component21">
+        <inertial>
+            <origin xyz="1.4090898048380041e-09 -3.2535507088482518e-09 0.044599997971269886" rpy="0.0 -0.0 0.0" />
+            <mass value="6.7233963282067295" />
+            <inertia ixx="0.010956805237582745" iyy="0.010956805237583245" izz="0.019417168595860734" ixy="-4.3216976490249204e-33" iyz="-5.607368611713793e-17" ixz="-1.3522991753733583e-33" />
+        </inertial>
+        <visual name="Component21_visual">
+            <origin xyz="1.4090898048380041e-09 -3.253550886483936e-09 0.06819999797126981" rpy="1.570796326794897 1.57079632679489 0" />
+            <geometry>
+                <mesh filename="package://arm_urdf/meshes/Component21.stl" scale="0.001 0.001 0.001" />
+            </geometry>
+        </visual>
+        <collision name="Component21_collision">
+            <origin xyz="1.4090898048380041e-09 -3.253550886483936e-09 0.06819999797126981" rpy="1.570796326794897 1.57079632679489 0" />
+            <geometry>
+                <mesh filename="package://arm_urdf/meshes/Component21.stl" scale="0.001 0.001 0.001" />
+            </geometry>
+        </collision>
+    </link>
+    <link name="Component22">
+        <inertial>
+            <origin xyz="1.4090898758922778e-09 -3.2535475469330776e-09 -0.044600002028730226" rpy="0.0 -0.0 0.0" />
+            <mass value="6.7233963282067295" />
+            <inertia ixx="0.01095680523758269" iyy="0.010956805237583356" izz="0.019417168595860568" ixy="-5.551115123125783e-17" iyz="-1.3364775223853718e-16" ixz="3.230809805085395e-32" />
+        </inertial>
+        <visual name="Component22_visual">
+            <origin xyz="1.4090898758922778e-09 -3.253547689041625e-09 -0.0210000020287303" rpy="1.570796326794897 1.5707963267948912 0" />
+            <geometry>
+                <mesh filename="package://arm_urdf/meshes/Component22.stl" scale="0.001 0.001 0.001" />
+            </geometry>
+        </visual>
+        <collision name="Component22_collision">
+            <origin xyz="1.4090898758922778e-09 -3.253547689041625e-09 -0.0210000020287303" rpy="1.570796326794897 1.5707963267948912 0" />
+            <geometry>
+                <mesh filename="package://arm_urdf/meshes/Component22.stl" scale="0.001 0.001 0.001" />
+            </geometry>
+        </collision>
+    </link>
+    <link name="Component23">
+        <inertial>
+            <origin xyz="1.4090897337837305e-09 -3.2535485239293393e-09 -0.07080000202872959" rpy="0.0 -0.0 0.0" />
+            <mass value="6.7233963282067295" />
+            <inertia ixx="0.010956805237582912" iyy="0.010956805237583467" izz="0.019417168595860734" ixy="-5.5511151231257765e-17" iyz="5.130125839607422e-18" ixz="1.1102230246251568e-16" />
+        </inertial>
+        <visual name="Component23_visual">
+            <origin xyz="1.4090897337837305e-09 -3.253548417347929e-09 -0.09440000202872952" rpy="1.5707963267948963 -1.5707963267948912 0" />
+            <geometry>
+                <mesh filename="package://arm_urdf/meshes/Component23.stl" scale="0.001 0.001 0.001" />
+            </geometry>
+        </visual>
+        <collision name="Component23_collision">
+            <origin xyz="1.4090897337837305e-09 -3.253548417347929e-09 -0.09440000202872952" rpy="1.5707963267948963 -1.5707963267948912 0" />
+            <geometry>
+                <mesh filename="package://arm_urdf/meshes/Component23.stl" scale="0.001 0.001 0.001" />
+            </geometry>
+        </collision>
+    </link>
+    <link name="long-v2">
+        <inertial>
+            <origin xyz="0.009999997971266881 0.001999998590900454 0.3773517377432081" rpy="0.0 -0.0 0.0" />
+            <mass value="1.0035470040377286" />
+            <inertia ixx="0.04728019585748308" iyy="0.0472801232304033" izz="8.152769985997343e-05" ixy="-6.38378239159465e-16" iyz="-1.4849232954361469e-15" ixz="-9.26342336171615e-16" />
+        </inertial>
+        <visual name="long-v2_visual">
+            <origin xyz="0.00999999797127173 0.001999998590902621 -0.8999999967464486" rpy="1.570796326794894 -6.31805127858374e-16 1.5707963267948972" />
+            <geometry>
+                <mesh filename="package://arm_urdf/meshes/long-v2.stl" scale="0.001 0.001 0.001" />
+            </geometry>
+        </visual>
+        <collision name="long-v2_collision">
+            <origin xyz="0.00999999797127173 0.001999998590902621 -0.8999999967464486" rpy="1.570796326794894 -6.31805127858374e-16 1.5707963267948972" />
+            <geometry>
+                <mesh filename="package://arm_urdf/meshes/long-v2.stl" scale="0.001 0.001 0.001" />
+            </geometry>
+        </collision>
+    </link>
+    <link name="depth_CamMount-v1">
+        <inertial>
+            <origin xyz="-0.010000400047506589 -0.008874522160693062 0.01856899713210183" rpy="1.0947644252537636e-47 -0.0 2.167227418503721e-47" />
+            <mass value="0.3638731014386725" />
+            <inertia ixx="0.00012703039538089484" iyy="0.0006733838995720831" izz="0.0005842583201846813" ixy="-2.013649249097471e-09" iyz="7.605648956632293e-06" ixz="4.2427877746841524e-10" />
+        </inertial>
+        <visual name="depth_CamMount-v1_visual">
+            <origin xyz="0.11400000040019924 -0.06568965261112218 0.002882962337094881" rpy="3.141592653589786 -0.7853981633974474 1.570796326795628" />
+            <geometry>
+                <mesh filename="package://arm_urdf/meshes/depth_CamMount-v1.stl" scale="0.001 0.001 0.001" />
+            </geometry>
+        </visual>
+        <collision name="depth_CamMount-v1_collision">
+            <origin xyz="0.11400000040019924 -0.06568965261112218 0.002882962337094881" rpy="3.141592653589786 -0.7853981633974474 1.570796326795628" />
+            <geometry>
+                <mesh filename="package://arm_urdf/meshes/depth_CamMount-v1.stl" scale="0.001 0.001 0.001" />
+            </geometry>
+        </collision>
+    </link>
+    <link name="depthCam-v1">
+        <inertial>
+            <origin xyz="-0.00935716369844542 0.00924907721198755 0.015605867277937656" rpy="-5.605193857299268e-45 -0.0 0.0" />
+            <mass value="1.3163395126511606" />
+            <inertia ixx="0.0030530914449512503" iyy="0.00025654140400710446" izz="0.0030520472296760026" ixy="9.36949828833633e-09" iyz="-3.302601715021724e-08" ixz="3.105331512459619e-05" />
+        </inertial>
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